File: kicad/esp32_project.kicad_sch (KiCad schematic)
At the start: 4 parts, among them U1 ESP32_DevKit_v1, U2 SHT31-D

Commit message: feat: IoT schema
Parts:
- added LAS1: KY-008, Connector:PinHeader_1x03_P2.54mm_Vertical, symbol Project_Parts:KY008_Laser
- added LDR1: LDR_Module, Connector:PinHeader_1x03_P2.54mm_Vertical, symbol Project_Parts:LDR_Module
Connections:
- net GND: now also LAS1.3 (GND), LDR1.2 (GND)
- net at AN1.4 (VCC), U1.1 (3V3), U2.5 (VDD): now also LAS1.2 (VCC), LDR1.1 (VCC)
- net at U1.22 (GPIO19): now also LAS1.1 (S)
- net at U1.5 (GPIO34): now also LDR1.3 (OUT)
Other:
- note added: "Deteksi keberadaan kabut"
- note added: "dari cahaya laser"
- note added: "lewat pembacaan sensor LDR"
- company: (none) -> Tim "Kata Ketua Buat Nama Tim Harus Diskusi Dulu"
- title: (none) -> Skema IoT - Kontrol Via Blynk
- moved on the sheet: AN1, U2

Commit message: feat: conditional activation
Connections:
- net +5V: now also AN1.4 (VCC)
- net at LAS1.2 (VCC), LDR1.1 (VCC), U1.1 (3V3)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: no longer AN1.4 (VCC)
Changed lines of the file:
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@@
-	)
-	(junction
-		(at 165.1 107.95)
-		(diameter 0)
-		(color 0 0 0 0)
 	)
 	(junction
@@
 		(pts
 			(xy 152.4 92.71) (xy 158.75 92.71)
-		)
-		(stroke
-			(width 0)
-			(type default)
-		)
-	)
-	(wire
-		(pts
-			(xy 165.1 107.95) (xy 171.45 107.95)
 		)
 		(stroke
@@
 		)
 	)
+	(junction
+		(at 181.61 88.9)
+		(diameter 0)
+		(color 0 0 0 0)
+	)
+	(wire
+		(pts
+			(xy 171.45 107.95) (xy 171.45 113.03)
+		)
+		(stroke
+			(width 0)
+			(type default)
+		)
+	)
+	(wire
+		(pts
+			(xy 171.45 113.03) (xy 126.99999999999999 113.03)
+		)
+		(stroke
+			(width 0)
+			(type default)
+		)
+	)
+	(junction
+		(at 127.0 113.03)
+		(diameter 0)
+		(color 0 0 0 0)
+	)
 	(sheet_instances
